File: documentation/zapojeni/horni.kicad_sch (KiCad schematic)
At the start: 29 parts

Commit message: jede celej spodek
Parts:
- R1, R2, R3: value 220R -> 1k
Changed lines of the file:
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@@
 	)
 	(junction
-		(at 275.59 26.67)
-		(diameter 0)
-		(color 0 0 0 0)
-	)
-	(junction
 		(at 20.32 81.28)
 		(diameter 0)
@@
 	(wire
 		(pts
-			(xy 269.24 26.67) (xy 275.59 26.67)
+			(xy 217.17 43.18) (xy 222.25 43.18)
 		)
 		(stroke
@@
 	(wire
 		(pts
-			(xy 217.17 43.18) (xy 222.25 43.18)
+			(xy 269.24 26.67) (xy 275.59 26.67)
 		)
 		(stroke
@@
 	(wire
 		(pts
-			(xy 278.13 26.67) (xy 275.59 26.67)
-		)
-		(stroke
-			(width 0)
-			(type default)
-		)
-	)
-	(wire
-		(pts
 			(xy 95.25 123.19) (xy 100.33 123.19)
 		)
@@
 			)
 		)
-		(property "Value" "220R"
+		(property "Value" "1k"
 			(at 207.01 22.86 90)
 			(effects
@@
 			)
 		)
-		(property "Value" "220R"
+		(property "Value" "1k"
 			(at 160.02 22.86 90)
 			(effects
@@
 			)
 		)
-		(property "Value" "220R"
+		(property "Value" "1k"
 			(at 251.46 22.86 90)
 			(effects
